File: MicroView.brd (EAGLE design)
At the start: 20.5 x 20.5 mm, 25 parts, among them J1 OLED_SCREEN, J2 MICROVIEW-16, J3 M03NS_SLIM, U1 MIC5205 3.3V, U2 SPX3819M5-L-5-0, U3 ATMEGA328P, Y1 16MHz

Commit message: v02 from SparkFun
Parts:
- removed J3: M03NS_SLIM, microView-temp:1X03_NS_SLIM
- removed Y1: 16MHz, SparkFun-FreqCtrl:RESONATOR-SMD
- added J4: M03NS_SLIM, microView-temp:1X03_NS_SLIM
- added R3, R4: 10K, SparkFun-Resistors:0603-RES
- added Y2: RESONATORSMD, microView-temp:RESONATOR-SMD
- moved C2 3.78 mm to (-9.14, -1.27), turned to 270 degrees
- moved U2 2.54 mm to (-6.35, 2.03)
- moved C4 2.04 mm to (-6.35, 4.32)
- moved C1 1.40 mm to (-6.35, 5.59), turned to 0 degrees
- moved C3 1.27 mm to (-6.35, -3.81)
- moved U1 1.27 mm to (-6.35, -1.27), turned to 270 degrees
- turned C10 to 90 degrees
Connections:
- new net D4/3.3V_EN: U1.3, U3.2
- new net D7/!RESET!: OLED1.12, R4.2, U3.11
- net 5V: now also C1.1, R3.2, U1.1
- net D10/SS: now also R3.1
- net D11/MOSI: now also J4.1; no longer J3.1
- net D12/MISO: now also J4.3; no longer J3.2, OLED1.12
- net D13/SCK: now also J4.2; no longer J3.3
- net GND: now also R4.1, Y2.2; no longer Y1.2
- net N$8: now also Y2.1; no longer Y1.1
- net N$9: now also Y2.3; no longer Y1.3
- net VIN: no longer C1.1, U1.1, U1.3
Routing:
- net VIN: track 25.6 -> 12.7 mm
- net 5V: track 32.8 -> 45.3 mm
- net D10/SS: track 10.8 -> 22.3 mm, vias 1 -> 2
- net D7/!RESET!: track 0.00 -> 11.1 mm, vias 0 -> 1
- net D12/MISO: track 14.5 -> 7.50 mm
- net D6: track 11.9 -> 6.36 mm
- net D5: track 7.98 -> 11.9 mm, vias 2 -> 1
- net D2: track 21.0 -> 18.7 mm
- net D4/3.3V_EN: track 0.00 -> 2.12 mm
- net 3.3V: track 10.8 -> 12.4 mm
- net D3: track 21.4 -> 19.9 mm
- net TXD: track 19.1 -> 17.7 mm
- net N$8: track 4.51 -> 5.42 mm
- net D11/MOSI: track 13.1 -> 12.2 mm
- net GND: track 15.4 -> 16.2 mm
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Other:
- board text removed: "v01"

Commit message: Production Final version V10
Parts:
- removed J4: M03NS_SLIM, microView-temp:1X03_NS_SLIM
- added TP1, TP2, TP3: (no value), SparkFun-Passives:PAD.03X.05
- R3, R4: value 10K -> 1k
- Y2: value RESONATORSMD -> 16MHz
- moved R3 14.0 mm to (7.62, 6.10), turned to 270 degrees
- moved C7 13.4 mm to (-6.35, 7.11), turned to 0 degrees
- moved R4 5.14 mm to (6.35, 6.10), turned to 270 degrees
- moved C1 4.57 mm to (-6.35, 1.02)
- moved C4 1.52 mm to (-6.35, 5.84)
- moved U2 1.27 mm to (-6.35, 3.30)
- moved C8 0.38 mm to (7.62, 2.16)
- moved C2 0.13 mm to (-9.14, -1.40)
Connections:
- new net D11: R4.2, TP3.P$1, U3.15
- new net D13: R3.2, TP2.P$1, U3.17
- net 5V: no longer R3.2
- net D10/SS: no longer R3.1
- net D11/MOSI: now also R4.1; no longer J4.1, U3.15
- net D12/MISO: now also TP1.P$1; no longer J4.3
- net D13/SCK: now also R3.1; no longer J4.2, U3.17
- net D7/!RESET!: no longer R4.2
- net GND: no longer R4.1
Routing:
- net D10/SS: track 22.3 -> 10.1 mm, vias 2 -> 1
- net D11: track 0.00 -> 6.55 mm, vias 0 -> 1
- net D12/MISO: track 7.50 -> 1.07 mm, vias 0 -> 1
- net D13: track 0.00 -> 5.47 mm, vias 0 -> 1
- net 5V: track 45.3 -> 39.9 mm
- net GND: track 16.2 -> 19.8 mm, vias 8 -> 9
- net D7/!RESET!: track 11.1 -> 8.35 mm
- net D13/SCK: track 14.0 -> 16.6 mm
- net D5: track 11.9 -> 9.52 mm
- net VIN: track 12.7 -> 14.3 mm
- net D11/MOSI: track 12.2 -> 13.2 mm
- net D6: track 6.36 -> 7.26 mm
- net C2N: track 5.94 -> 6.64 mm
