File: MicroView.sch (EAGLE design)
At the start: 25 parts, among them J1 OLED_SCREEN, J2 MICROVIEW-16, J3 M03NS_SLIM, U1 MIC5205 3.3V, U2 SPX3819M5-L-5-0, U3 ATMEGA328P, Y1 16MHz

Commit message: v02 from SparkFun
Parts:
- removed J3: M03NS_SLIM, microView-temp:M03NS_SLIM
- removed Y1: 16MHz, SparkFun-FreqCtrl:RESONATOR16MHZ
- added J4: M03NS_SLIM, microView-temp:M03NS_SLIM
- added R3, R4: 10K, SparkFun-Resistors:10KOHM1/10W1%(0603)0603
- added Y2: RESONATORSMD, microView-temp:RESONATORSMD
Connections:
- new net D4/3.3V_EN: U1.EN, U3.PD4(XCK/T0)
- new net D7/!RESET!: OLED1.!RESET!, R4.2, U3.PD7(AIN1)
- net 5V: now also C1.1, R3.2, U1.IN
- net D10/SS: now also R3.1
- net D11/MOSI: now also J4.1; no longer J3.1
- net D12/MISO: now also J4.3; no longer J3.2, OLED1.!RESET!
- net D13/SCK: now also J4.2; no longer J3.3
- net GND: now also R4.1, Y2.2; no longer Y1.2
- net N$8: now also Y2.1; no longer Y1.1
- net N$9: now also Y2.3; no longer Y1.3
- net VIN: no longer C1.1, U1.EN, U1.IN
Other:
- note added: "ATmega328"
- note added: "Headers"
- note added: "OLED"
- note added: "Voltage Regulators"
- note added: "v02"
- note removed: "v01"
- moved on the sheet: C1, C2, C3, C4, U1, U2

Commit message: Production Final version V10
Parts:
- removed J4: M03NS_SLIM, microView-temp:M03NS_SLIM
- added TP1, TP2, TP3: TEST-POINT3X5, SparkFun-Passives:TEST-POINT3X5
- R3, R4: value 10K -> 1k
- Y2: value RESONATORSMD -> 16MHz
Connections:
- new net D11: R4.2, TP3.1, U3.PB3(MOSI/OC2)
- new net D13: R3.2, TP2.1, U3.PB5(SCK)
- net 5V: no longer R3.2
- net D10/SS: no longer R3.1
- net D11/MOSI: now also R4.1; no longer J4.1, U3.PB3(MOSI/OC2)
- net D12/MISO: now also TP1.1; no longer J4.3
- net D13/SCK: now also R3.1; no longer J4.2, U3.PB5(SCK)
- net D7/!RESET!: no longer R4.2
- net GND: no longer R4.1
Other:
- note added: "v10"
- note removed: "v02"
- moved on the sheet: C1, R3, R4
